File: Hardware/MicroBit_Breakout.sch (EAGLE design)
At the start: 3 parts, among them J1 M22LOCK, X1 EDGE-80PTH-RA

Commit message: Layout complete
Parts:
- added FD1, FD2: FIDUCIAL1X2, SparkFun-Aesthetics:FIDUCIAL1X2
- added H1, H2: STAND-OFF, SparkFun-Electromechanical:STAND-OFF
- added LOGO1: SFE_LOGO_FLAME.1_INCH, SparkFun-Aesthetics:SFE_LOGO_FLAME.1_INCH
- added LOGO3: OSHW-LOGOS, SparkFun-Aesthetics:OSHW-LOGOS
Connections:
- net N$1 renamed GND
Changed lines of the file:
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@@
 <part name="X1" library="SparkFun-Connectors" deviceset="EDGE-80" device="PTH-RA"/>
 <part name="J1" library="SparkFun-Connectors" deviceset="M22" device="LOCK"/>
+<part name="FD1" library="SparkFun-Aesthetics" deviceset="FIDUCIAL" device="1X2"/>
+<part name="FD2" library="SparkFun-Aesthetics" deviceset="FIDUCIAL" device="1X2"/>
+<part name="H1" library="SparkFun-Electromechanical" deviceset="STAND-OFF" device=""/>
+<part name="H2" library="SparkFun-Electromechanical" deviceset="STAND-OFF" device=""/>
+<part name="LOGO1" library="SparkFun-Aesthetics" deviceset="SFE_LOGO_FLAME" device=".1_INCH"/>
+<part name="LOGO3" library="SparkFun-Aesthetics" deviceset="OSHW-LOGO" device="S"/>
 </parts>
 <sheets>
@@
 <instance part="X1" gate="G$1" x="127" y="106.68"/>
 <instance part="J1" gate="G$1" x="50.8" y="93.98" rot="MR180"/>
+<instance part="FD1" gate="G$1" x="243.84" y="33.02"/>
+<instance part="FD2" gate="G$1" x="243.84" y="27.94"/>
+<instance part="H1" gate="G$1" x="238.76" y="33.02"/>
+<instance part="H2" gate="G$1" x="238.76" y="27.94"/>
+<instance part="LOGO1" gate="G$1" x="129.54" y="22.86"/>
+<instance part="LOGO3" gate="G$1" x="132.08" y="12.7"/>
 </instances>
 <busses>
 </busses>
 <nets>
-<net name="N$1" class="0">
+<net name="GND" class="0">
 <segment>
 <pinref part="X1" gate="G$1" pin="A1"/>
